Commit message: URDF rotation bug fix

File: demo/resources/human.urdf (robot description, URDF)
Before this commit: robot human, 24 links, 23 joints
Joints:
- joint ArmL: origin xyz=0.1848 -0.0185001 0.0028 rpy=0 0 0 -> xyz=0.1848 -0.0185001 0.0028 rpy=-0 0 -0
- joint ArmR: origin xyz=-0.1848 -0.0185001 0.0028 rpy=0 0 0 -> xyz=-0.1848 -0.0185001 0.0028 rpy=-0 0 -0
- joint FemurL: origin xyz=0.0903 -0.0472 0.0192 rpy=0 0 0 -> xyz=0.0903 -0.0472 0.0192 rpy=-0 0 -0
- joint FemurR: origin xyz=-0.0903 -0.0472 0.0192 rpy=0 0 0 -> xyz=-0.0903 -0.0472 0.0192 rpy=-0 0 -0
- joint FootPinkyL: origin xyz=0.0427 -0.0634 0.0913 rpy=0 0 0 -> xyz=0.0427 -0.0634 0.0913 rpy=-0 0 -0
- joint FootPinkyR: origin xyz=-0.0427 -0.0634 0.0913 rpy=0 0 0 -> xyz=-0.0427 -0.0634 0.0913 rpy=-0 0 -0
- joint FootThumbL: origin xyz=-0.00189999 -0.0575 0.1111 rpy=0 0 0 -> xyz=-0.00189999 -0.0575 0.1111 rpy=-0 0 -0
- joint FootThumbR: origin xyz=0.00189999 -0.0575 0.1111 rpy=0 0 0 -> xyz=0.00189999 -0.0575 0.1111 rpy=-0 0 -0
- joint ForeArmL: origin xyz=0.3239 0.0257001 0.0248 rpy=0 0 0 -> xyz=0.3239 0.0257001 0.0248 rpy=-0 0 -0
- joint ForeArmR: origin xyz=-0.3239 0.0257001 0.0248 rpy=0 0 0 -> xyz=-0.3239 0.0257001 0.0248 rpy=-0 0 -0
- joint HandL: origin xyz=0.2868 0.00870001 0.0299 rpy=0 0 0 -> xyz=0.2868 0.00870001 0.0299 rpy=-0 0 -0
- joint HandR: origin xyz=-0.2868 0.00829995 0.0299 rpy=0 0 0 -> xyz=-0.2868 0.00829995 0.0299 rpy=-0 0 -0
- joint Head: origin xyz=0 0.0807999 0.035 rpy=0 0 0 -> xyz=0 0.0807999 0.035 rpy=-0 0 -0
- joint Neck: origin xyz=0 0.3083 0.0062 rpy=0 0 0 -> xyz=0 0.3083 0.0062 rpy=-0 0 -0
- joint Pelvis: origin xyz=0 0.9809 -0.0308 rpy=0 0 0 -> xyz=0 0.9809 -0.0308 rpy=-0 0 -0
- joint ShoulderL: origin xyz=0.0147 0.2774 0.0117 rpy=0 0 0 -> xyz=0.0147 0.2774 0.0117 rpy=-0 0 -0
- joint ShoulderR: origin xyz=-0.0147 0.2774 0.0117 rpy=0 0 0 -> xyz=-0.0147 0.2774 0.0117 rpy=-0 0 -0
- joint Spine: origin xyz=0 0.0866 -0.0126 rpy=0 0 0 -> xyz=0 0.0866 -0.0126 rpy=-0 0 -0
- joint TalusL: origin xyz=-0.0195 -0.4611 -0.0316 rpy=0 0 0 -> xyz=-0.0195 -0.4611 -0.0316 rpy=-0 0 -0
- joint TalusR: origin xyz=0.0195 -0.4611 -0.0316 rpy=0 0 0 -> xyz=0.0195 -0.4611 -0.0316 rpy=-0 0 -0
- joint TibiaL: origin xyz=0.0092 -0.395 0.0013 rpy=0 0 0 -> xyz=0.0092 -0.395 0.0013 rpy=-0 0 -0
- joint TibiaR: origin xyz=-0.0092 -0.395 0.0013 rpy=0 0 0 -> xyz=-0.0092 -0.395 0.0013 rpy=-0 0 -0
- joint Torso: origin xyz=0 0.1086 -0.0064 rpy=0 0 0 -> xyz=0 0.1086 -0.0064 rpy=-0 0 -0

Commit message: Initial test impl (not working yet...)

File: demo/resources/human.urdf (robot description, URDF)
Before this commit: robot human, 24 links, 23 joints
Joints:
- joint Head: type revolute -> spherical
- joint Pelvis: origin xyz=0 0.9809 -0.0308 rpy=-0 0 -0 -> xyz=0 0 0 rpy=-0 0 -0
